File: _Kicad/keyboard.kicad_pcb (KiCad board)
At the start: 2 copper layers, 372.1 x 134.6 mm, 189 parts, among them J2 Conn_02x20_Top_Bottom

Commit message: fix controller pins and orientation painnnnnnnnnn
Connections:
- J2 pad 10: /12x8/COL2 -> /12x8/ROT3A
- J2 pad 11: unconnected-(J2-Pin_11-Pad11) -> /12x8/COL5
- J2 pad 12: /12x8/COL3 -> /12x8/COL4
- J2 pad 13: /12x8/COL4 -> /12x8/COL3
- J2 pad 14: /12x8/COL5 -> unconnected-(J2-Pin_14-Pad14)
- J2 pad 15: /12x8/ROT3A -> /12x8/COL2
- J2 pad 16: unconnected-(J2-Pin_16-Pad16) -> /12x8/COL1
- J2 pad 17: /12x8/COL6 -> /12x8/ROT1A
- J2 pad 18: /12x8/COL7 -> /12x8/ROT1B
- J2 pad 19: /12x8/COL8 -> /12x8/ROT2A
- J2 pad 2: unconnected-(J2-Pin_2-Pad2) -> /12x8/COL8
- J2 pad 21: /12x8/ROW2 -> /12x8/ROT2B
- J2 pad 25: /12x8/ROW3 -> /12x8/ROW2
- J2 pad 26: unconnected-(J2-Pin_26-Pad26) -> /12x8/ROW4
- J2 pad 27: unconnected-(J2-Pin_27-Pad27) -> /12x8/ROW6
- J2 pad 28: unconnected-(J2-Pin_28-Pad28) -> /12x8/ROW1
- J2 pad 29: unconnected-(J2-Pin_29-Pad29) -> /12x8/ROW3
- J2 pad 3: unconnected-(J2-Pin_3-Pad3) -> /12x8/COL7
- J2 pad 30: /12x8/ROW5 -> unconnected-(J2-Pin_30-Pad30)
- J2 pad 31: /12x8/ROW7 -> unconnected-(J2-Pin_31-Pad31)
- J2 pad 32: /12x8/ROW9 -> unconnected-(J2-Pin_32-Pad32)
- J2 pad 33: /12x8/ROW11 -> unconnected-(J2-Pin_33-Pad33)
- J2 pad 38: unconnected-(J2-Pin_38-Pad38) -> /12x8/ROW5
- J2 pad 39: unconnected-(J2-Pin_39-Pad39) -> /12x8/ROW7
- J2 pad 4: /12x8/ROT2B -> /12x8/COL6
- J2 pad 40: unconnected-(J2-Pin_40-Pad40) -> /12x8/ROW9
- J2 pad 7: /12x8/ROT1B -> unconnected-(J2-Pin_7-Pad7)
