File: _Kicad/untitled.kicad_sch (KiCad schematic)
At the start: 189 parts, among them J2 Conn_02x20_Top_Bottom

Commit message: fix controller pins and orientation painnnnnnnnnn
Connections:
- net COL1: now also J2.16 (Pin_16); no longer J2.9 (Pin_9)
- net COL2: now also J2.15 (Pin_15); no longer J2.10 (Pin_10)
- net COL3: now also J2.13 (Pin_13); no longer J2.12 (Pin_12)
- net COL4: now also J2.12 (Pin_12); no longer J2.13 (Pin_13)
- net COL5: now also J2.11 (Pin_11); no longer J2.14 (Pin_14)
- net COL6: now also J2.4 (Pin_4); no longer J2.17 (Pin_17)
- net COL7: now also J2.3 (Pin_3); no longer J2.18 (Pin_18)
- net COL8: now also J2.2 (Pin_2); no longer J2.19 (Pin_19)
- net ROT1A: now also J2.17 (Pin_17); no longer J2.8 (Pin_8)
- net ROT1B: now also J2.18 (Pin_18); no longer J2.7 (Pin_7)
- net ROT2A: now also J2.19 (Pin_19); no longer J2.6 (Pin_6)
- net ROT2B: now also J2.21 (Pin_21); no longer J2.4 (Pin_4)
- net ROT3A: now also J2.10 (Pin_10); no longer J2.15 (Pin_15)
- net ROT3B: now also J2.46 (Pin_46); no longer J2.37 (Pin_37)
- net ROW1: now also J2.28 (Pin_28); no longer J2.24 (Pin_24)
- net ROW10: now also J2.43 (Pin_43); no longer J2.35 (Pin_35)
- net ROW11: now also J2.41 (Pin_41); no longer J2.33 (Pin_33)
- net ROW12: now also J2.45 (Pin_45); no longer J2.36 (Pin_36)
- net ROW2: now also J2.25 (Pin_25); no longer J2.21 (Pin_21)
- net ROW3: now also J2.29 (Pin_29); no longer J2.25 (Pin_25)
- net ROW4: now also J2.26 (Pin_26); no longer J2.22 (Pin_22)
- net ROW5: now also J2.38 (Pin_38); no longer J2.30 (Pin_30)
- net ROW6: now also J2.27 (Pin_27); no longer J2.23 (Pin_23)
- net ROW7: now also J2.39 (Pin_39); no longer J2.31 (Pin_31)
- net ROW8: now also J2.42 (Pin_42); no longer J2.34 (Pin_34)
- net ROW9: now also J2.40 (Pin_40); no longer J2.32 (Pin_32)
Changed lines of the file:
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@@
 	(symbol
 		(lib_id "Connector_Generic:Conn_02x20_Top_Bottom")
-		(at 439.42 88.9 0)
-		(mirror y)
+		(at 436.88 88.9 0)
 		(unit 1)
 		(exclude_from_sim no)
@@
 		)
 		(property "Footprint" "my library:blackpill"
-			(at 439.42 88.9 0)
+			(at 436.88 88.9 0)
 			(effects
 				(font
@@
 		)
 		(property "Datasheet" "~"
-			(at 439.42 88.9 0)
+			(at 436.88 88.9 0)
 			(effects
 				(font
@@
 		)
 		(property "Description" "Generic connector, double row, 02x20, top/bottom pin numbering scheme (row 1: 1...pins_per_row, row2: pins_per_row+1 ... num_pins), script generated (kicad-library-utils/schlib/autogen/connector/)"
-			(at 439.42 88.9 0)
+			(at 436.88 88.9 0)
 			(effects
 				(font
@@
 		(pin "40"
 		)
-		(pin "9"
+		(pin "42"
 		)
-		(pin "6"
+		(pin "5v"
 		)
 		(pin "7"
@@
 		(pin "2"
 		)
-		(pin "5"
+		(pin "3v3"
 		)
-		(pin "34"
+		(pin "G"
 		)
-		(pin "37"
+		(pin "G"
 		)
 		(pin "21"
@@
 		(pin "39"
 		)
-		(pin "8"
+		(pin "45"
 		)
 		(pin "13"
@@
 		(pin "3"
 		)
-		(pin "36"
+		(pin "43"
 		)
 		(pin "26"
@@
 		(pin "1"
 		)
-		(pin "35"
+		(pin "5v"
 		)
 		(pin "19"
@@
 		(pin "11"
 		)
-		(pin "24"
+		(pin "46"
 		)
-		(pin "23"
+		(pin "41"
 		)
 		(pin "28"
@@
 		(pin "15"
 		)
-		(pin "22"
+		(pin "3v3"
 		)
 		(pin "27"
